File: EthercatIOBoard/encoderIn.kicad_sch (KiCad schematic)
At the start: 12 parts, among them J12 Conn_02x04_Odd_Even, U31 SP3485EN, U32 SP3485EN, U33 SP3485EN

Commit message: small improvments
Parts:
- added R226, R231, R235, R236, R243, R244: 12k, Resistor_SMD:R_0402_1005Metric, symbol Device:R
- R146, R147, R148: value 120 -> 1.5k
Connections:
- net A_H: now also R226.2
- net A_L: now also R231.1
- net B_H: now also R235.2
- net B_L: now also R236.1
- net GND: now also R231.2, R236.2, R244.2
- net Z_H: now also R243.2
- net Z_L: now also R244.1
- net at C126.2, C127.2, C128.2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: now also R226.1, R235.1, R243.1
Other:
- moved on the sheet: C126, C127, R145, R147, R148, U32, U33
