File: EthercatIOBoard/EthercatIOBoard.kicad_sch (KiCad schematic)
At the start: 5 parts, among them J1 Conn_01x03

Commit message: some cleanup
Other:
- sheet Ethercat1 ports: added EE_SCL, EE_SDA; removed none
