File: EthercatIOBoard/ethercat2.kicad_sch (KiCad schematic)
At the start: 62 parts, among them J18 RJ45_Hanrun_HR911105A_Horizon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, J2 RJ45_Hanrun_HR911105A_Horizon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, U2 AX58100, U3 24LC512, U4 TLV71312PDBV, Y1 25Mhz

Commit message: some cleanup
Connections:
- net SCL renamed EE_SCL
- net SDA renamed EE_SDA
Other:
- moved on the sheet: R173, R174, U3
